Commit message: compute a new plan, still fails in the simulation

File: solvers/trajectoryOptimization/dev/cinderblock.urdf (robot description, URDF)
Before this commit: robot CinderBlock, 1 links, 0 joints
Links:
- link block: geometry collision box size=0.397 3 0.29; visual box size=0.397 3 0.29
