Commit message: start to test analytical IK against global IK

File: drake/examples/IRB140/urdf/irb_140_shift.urdf (robot description, URDF)
Before this commit: robot IRB140_-_M2004C_Complete_base.SLDASM, 7 links, 6 joints
Links:
- link base_link: geometry visual mesh filename=./meshes/base_link.stl
- link link_1: geometry visual mesh filename=./meshes/link1.stl
- link link_2: geometry visual mesh filename=./meshes/link2.stl
- link link_3: geometry visual mesh filename=./meshes/link3.stl
- link link_4: geometry visual mesh filename=./meshes/link4.stl
- link link_5: geometry visual mesh filename=./meshes/link5.stl
- link link_6: geometry visual mesh filename=./meshes/link6.stl
