Commit message: collision avoidance works for the demo

File: drake/manipulation/models/objects/coffee_mug/urdf/coffee_mug.urdf (robot description, URDF)
Before this commit: robot coffee_mug, 1 links, 0 joints
Links:
- link coffee_mug: geometry collision cylinder length=0.05 radius=0.07; visual mesh filename=../meshes/coffee_mug.obj
