Commit message: Get the key frames

File: drake/examples/kuka_iiwa_arm/dev/dual_arms_manipulation/box.urdf (robot description, URDF)
Before this commit: robot box, 1 links, 0 joints
Links:
- link box: geometry collision box size=0.56 0.56 0.56; visual box size=0.56 0.56 0.56

File: drake/manipulation/models/iiwa_description/urdf/dual_iiwa14_polytope_collision.urdf (robot description, URDF)
Before this commit: robot dual_iiwa14, 21 links, 19 joints
Joints:
- joint left_iiwa_base_joint: origin xyz=0 1.56 0 rpy=0 0 0 -> xyz=0 1.04 0 rpy=0 0 0
