Commit message: Plan the key frames for the whole rotating motion

File: drake/manipulation/models/iiwa_description/urdf/dual_iiwa14_polytope_collision.urdf (robot description, URDF)
Before this commit: robot dual_iiwa14, 21 links, 19 joints
Joints:
- joint left_iiwa_base_joint: origin xyz=0 1.04 0 rpy=0 0 0 -> xyz=0 0.96 0 rpy=0 0 0
