Commit message: Added object to manipulate. Added binding for setting penetration allowance (altho currently unused).

File: examples/2d_gripper/planar_gripper.xacro (robot description, xacro)
@@ -12,6 +12,6 @@
     <xacro:property name="l2_inertia" value="0.0083" />
     <xacro:property name="tip_radius" value="0.008" />
-    <xacro:property name="config_radius" value="0.18" />
-    <xacro:property name="config_angle" value="2.1" />
+    <!--<xacro:property name="config_radius" value="0.18" />-->
+    <!--<xacro:property name="config_angle" value="2.1" />-->
     <xacro:macro name="finger" params="fnum">
       <link name="finger${fnum}_base">

Commit message: Converts prismatic gripper to revolute gripper and updates the simulation.

File: examples/2d_gripper/planar_gripper.xacro (robot description, xacro)
@@ -2,14 +2,15 @@
 <sdf xmlns:xacro="http://www.ros.org/wiki/xacro" version='1.6'>
   <model name='planar_gripper'>
-    <xacro:property name="base_dim" value=".04" />
-    <xacro:property name="l1_length" value="0.1" />
-    <xacro:property name="l1_radius" value="0.005" />
+    <xacro:property name="base_dim" value=".08" />
+    <xacro:property name="l1_length" value="0.07" />
+    <xacro:property name="l1_radius" value="0.011" />
     <xacro:property name="l1_mass" value="0.1" />
     <xacro:property name="l1_inertia" value="0.0083" />
-    <xacro:property name="l2_length" value="0.1" />
-    <xacro:property name="l2_radius" value="0.005" />
+    <xacro:property name="l2_length" value="0.07" />
+    <xacro:property name="l2_radius" value="0.011" />
     <xacro:property name="l2_mass" value="0.1" />
     <xacro:property name="l2_inertia" value="0.0083" />
-    <xacro:property name="tip_radius" value="0.008" />
+    <xacro:property name="sensor_stack_len" value="0.001" />
+    <xacro:property name="tip_radius" value="0.015" />
     <!--<xacro:property name="config_radius" value="0.18" />-->
     <!--<xacro:property name="config_angle" value="2.1" />-->
@@ -47,5 +48,16 @@
           </geometry>
           <material>
-            <diffuse>0 1 0 1</diffuse>
+            <diffuse>1 0 0 1</diffuse>
+          </material>
+        </visual>
+        <visual name='link1_joint_visual'>
+          <pose>0 0 -${l1_length} 0 0 0</pose>
+          <geometry>
+            <sphere>
+              <radius>${l1_radius*1.2}</radius>
+            </sphere>
+          </geometry>
+          <material>
+            <diffuse>.1 .1 .1 1</diffuse>
           </material>
         </visual>
@@ -71,5 +83,5 @@
         <!-- The origin of the Link2 frame is defined to be coincident with
        the origin of the x-z plane in the elbow joint frame. -->
-        <pose>0 0 -${l1_length/2} 0 0 0</pose>
+        <pose>0 0 -${l1_length} 0 0 0</pose>
         <inertial>
           <pose>0 0 -${l2_length/2} 0 0 0</pose>
@@ -96,14 +108,25 @@
           </material>
         </visual>
-        <collision name='Link2_pad_collision'>
-          <pose>0 0 -${l2_length} 0 0 0</pose>
+        <visual name='link2_sensor'>
+          <pose>0 0 -${l2_length + sensor_stack_len} 0 0 0</pose>
           <geometry>
             <sphere>
-              <radius>0.008</radius>
+              <radius>${l2_radius}</radius>
+            </sphere>
+          </geometry>
+          <material>
+            <diffuse>.1 .1 .1 1</diffuse>
+          </material>
+        </visual>
+        <collision name='link2_pad_collision'>
+          <pose>0 0 -${l2_length + sensor_stack_len + tip_radius} 0 0 0</pose>
+          <geometry>
+            <sphere>
+              <radius>${tip_radius}</radius>
             </sphere>
           </geometry>
         </collision>
-        <visual name='Link2_pad_visual'>
-          <pose>0 0 -${l2_length} 0 0 0</pose>
+        <visual name='link2_pad_visual'>
+          <pose>0 0 -${l2_length + sensor_stack_len + tip_radius} 0 0 0</pose>
           <geometry>
             <sphere>
@@ -112,9 +135,9 @@
           </geometry>
           <material>
-            <diffuse>0 0 1 1</diffuse>
+            <diffuse>1 1 1 1</diffuse>
           </material>
         </visual>
       </link>
-      <joint name='finger${fnum}_ElbowJoint' type='prismatic'>
+      <joint name='finger${fnum}_ElbowJoint' type='revolute'>
         <parent>finger${fnum}_link1</parent>
         <child>finger${fnum}_link2</child>
@@ -122,11 +145,11 @@
         <pose>0 0 0 0 0 0</pose>
         <axis>
-          <xyz>0 0 1</xyz>
+          <xyz>1 0 0</xyz>
           <limit>
             <effort>100</effort>
             <!-- No limit provided. sdformat defaults to -1, which we parse as
                  an actuated joint. -->
-            <lower>-${l1_length/2}</lower>
-            <upper>${l1_length/2}</upper>
+            <lower>-1.57</lower>
+            <upper>1.57</upper>
           </limit>
           <dynamics>
