Commit message: adding test.cc and test2.cc

File: manipulation/models/iiwa_description/urdf/iiwa14_spheres_collision.urdf (robot description, URDF)
Before this commit: robot iiwa14, 11 links, 10 joints
Links:
- link iiwa_link_5: geometry visual mesh filename=../meshes/visual/band.obj; visual mesh filename=../meshes/visual/kuka.obj
