Commit message: Rebase on master. Change the dimension of the planar gripper to match with the hardware.

File: examples/planar_gripper/planar_gripper.xacro (robot description, xacro)
@@ -3,9 +3,9 @@
   <model name='planar_gripper'>
     <xacro:property name="base_dim" value=".08" />
-    <xacro:property name="l1_length" value="0.07" />
+    <xacro:property name="l1_length" value="0.085" />
     <xacro:property name="l1_radius" value="0.011" />
     <xacro:property name="l1_mass" value="0.1" />
     <xacro:property name="l1_inertia" value="0.0083" />
-    <xacro:property name="l2_length" value="0.07" />
+    <xacro:property name="l2_length" value="0.0563" />
     <xacro:property name="l2_radius" value="0.011" />
     <xacro:property name="l2_mass" value="0.1" />
