Commit message: Updated inertias to match hardware, including reflected motor-rotor inertia. Had to retune controller.

File: examples/planar_gripper/planar_finger.xacro (robot description, xacro)
@@ -6,11 +6,20 @@
     <xacro:property name="base_dim" value=".08" />
     <xacro:property name="l1_length" value="0.085" />
+    <xacro:property name="l1_COM" value="0.03811" />
     <xacro:property name="l1_radius" value="0.011" />
-    <xacro:property name="l1_mass" value="0.1" />
-    <xacro:property name="l1_inertia" value="0.0083" />
+    <xacro:property name="l1_mass" value="0.449" />
+    <xacro:property name="l1_xx_inertia" value="0.000200329" />
+    <xacro:property name="l1_yy_inertia" value="0.000774354" />
+    <xacro:property name="l1_zz_inertia" value="0.0006529" />
+    <xacro:property name="l1_xz_inertia" value="0.000028883" />
     <xacro:property name="l2_length" value="0.040" />
     <xacro:property name="l2_radius" value="0.011" />
-    <xacro:property name="l2_mass" value="0.1" />
-    <xacro:property name="l2_inertia" value="0.0083" />
+    <xacro:property name="l2_mass" value="0.104" />
+    <xacro:property name="l2_xx_inertia" value="0.000078462" />
+    <xacro:property name="l2_yy_inertia" value="0.000083214" />
+    <xacro:property name="l2_zz_inertia" value="0.000012773" />
+    <xacro:property name="l2_xz_inertia" value="0.000006523" />
+    <xacro:property name="shaft_inertia" value="0.0006" />
+    <xacro:property name="N" value="50" />
     <xacro:property name="sensor_length" value="0.005" />
     <xacro:property name="sensor_width" value="0.02" />
@@ -40,6 +49,10 @@
           <mass>${l1_mass}</mass>
           <inertia>
-            <ixx>${l1_inertia}</ixx><iyy>${l1_inertia}</iyy><izz>5e-7</izz>
-            <ixy>0</ixy><ixz>0</ixz><iyz>0</iyz>
+            <ixx>${l1_xx_inertia + (shaft_inertia * N * N) + (l1_mass * l1_length/2)}</ixx>
+            <iyy>${l1_yy_inertia + (shaft_inertia * N * N) + (l1_mass * l1_length/2)}</iyy>
+            <izz>${l1_zz_inertia}</izz>
+            <ixz>${l1_xz_inertia}</ixz>
+            <ixy>0</ixy>
+            <iyz>0</iyz>
           </inertia>
         </inertial>
@@ -92,6 +105,10 @@
           <mass>${l2_mass}</mass>
           <inertia>
-            <ixx>${l2_inertia}</ixx><iyy>${l2_inertia}</iyy><izz>5e-7</izz>
-            <ixy>0</ixy><ixz>0</ixz><iyz>0</iyz>
+            <ixx>${l2_xx_inertia  + (shaft_inertia * N * N) + (l1_mass * (l2_length + sensor_length + tip_adapter_length + tip_cylinder_length)/2)}</ixx>
+            <iyy>${l2_yy_inertia  + (shaft_inertia * N * N) + (l1_mass * (l2_length + sensor_length + tip_adapter_length + tip_cylinder_length)/2)}</iyy>
+            <izz>${l2_zz_inertia}</izz>
+            <ixz>${l2_xz_inertia}</ixz>
+            <ixy>0</ixy>
+            <iyz>0</iyz>
           </inertia>
         </inertial>
