Commit message: C iris pinball iiwa example (#45)
* rename sos_iris to C_iris and begin consolidating notebooks. Notebooks currently broken

* transfer IrisInRationalSpace back over

* checkpoint ready to debug snopt iris in t space

* just had to change how you were seeding

* transfer to desktop

* building of new iris file works but looks wrong on the pinball iiwa example

* finalized update to iris methods to include iris in rational cspace

* restore sos_iris_certifier folder for merg with C_Iris

* fixed gradient issue per https://github.com/RobotLocomotion/drake/pull/17003

* rename sos_iris to C_iris and begin consolidating notebooks. Notebooks currently broken

* add some hpolyhedron methods (#41)

* add some hpolyhedron methods

* fix lint issues in hpolyhedron

* add in the bindings for the Hpolyhedron methods

* updated names

* remove spurious file refs in bindings

* checkpoint

* add assets needed to make pinball iiwa example work up to snopt iris

* checkpoint

* update pinball iiwa to solve cleanly for one region. Deomnstrate some numerical issues

* add pinball iiwa example

* add pinball iiwa example and fix problem in HPolyhedron

* fixed some comments

* remove notebook outputs

* Delete C_Iris_Examples/__pycache__ directory

* moved shelves into model folder

* Merge branch 'C_Iris' of https://github.com/AlexandreAmice/drake into C_Iris_pinball_iiwa_example

* tweak some linting

File: C_Iris_Examples/assets/box_small.urdf (robot description, URDF)
Before this commit: robot box_scene, 5 links, 4 joints
Links:
- link box1: geometry collision box size=0.4 0.1 2.1; visual box size=0.4 0.1 2.1
- link box2: geometry collision box size=0.4 0.1 1.5; visual box size=0.4 0.1 1.5
- link box3: geometry collision box size=0.4 0.1 2.1; visual box size=0.4 0.1 2.1
- link box4: geometry collision box size=0.4 0.1 1.5; visual box size=0.4 0.1 1.5
Joints:
- joint jbox1: origin xyz=0 -0.55 -0.05 rpy=1.5707 0 0 -> xyz=0 0 -0.05 rpy=1.5707 0 0
- joint jbox2: origin xyz=0 0.6 1.0 rpy=0 0 0 -> xyz=0 1.0 .75 rpy=0 0 0
- joint jbox3: origin xyz=0 -0.55 2.0 rpy=1.5707 0 0 -> xyz=0 0 1.55 rpy=1.5707 0 0
- joint jbox4: origin xyz=0 -1.7 1.0 rpy=0 0 0 -> xyz=0 -1 .75 rpy=0 0 0
